File: Hardware/fatigue.kicad_sch (KiCad schematic)
At the start: 0 parts

Commit message: The fatigue machine PCB is really born
Parts:
- added C2, C3, C4, C5, C6, C7: C, symbol Device:C
- added J1: GPIO, Connector_PinSocket_2.54mm:PinSocket_2x20_P2.54mm_Vertical, symbol Connector_Generic:Conn_02x20_Odd_Even
- added U1: ADS1256IDBR, 1Personal:IC_ADC_ADS1256IDBR, symbol Custom:ADS1256IDBR
- added Y1: Crystal 8 MHz, symbol Device:Crystal
Connections:
- new net: C3.1, U1.18 (XTAL2), Y1.2
- new net: C2.1, U1.19 (XTAL1/CLKIN), Y1.1
- new net +3V3: C6.1, C7.1, J1.1 (Pin_1), J1.17 (Pin_17), U1.16 (DVDD)
- new net +5V: C4.1, C5.1, J1.2 (Pin_2), J1.4 (Pin_4), U1.1 (AVDD)
- new net GND: C2.2, C3.2, C4.2, C5.2, C6.2, C7.2, J1.14 (Pin_14), J1.20 (Pin_20), J1.25 (Pin_25), J1.30 (Pin_30), J1.34 (Pin_34), J1.39 (Pin_39), J1.6 (Pin_6), J1.9 (Pin_9), U1.17 (DGND), U1.2 (AGND)
- new net GPIO10/SPI0.MOSI: J1.19 (Pin_19), U1.23 (DIN)
- new net GPIO11/SPI0.SCLK: J1.23 (Pin_23), U1.24 (SCLK)
- new net GPIO12/PWM0: J1.32 (Pin_32)
- new net GPIO13/PWM1: J1.33 (Pin_33)
- new net GPIO14/TXD0: J1.8 (Pin_8)
- new net GPIO15/RXD0: J1.10 (Pin_10)
- new net GPIO16: J1.36 (Pin_36)
- new net GPIO17: J1.11 (Pin_11)
- new net GPIO18/PCM.CLK: J1.12 (Pin_12)
- new net GPIO19/PCM.FS: J1.35 (Pin_35)
- new net GPIO20/PCM.DIN: J1.38 (Pin_38)
- new net GPIO21/PCM.DOUT: J1.40 (Pin_40)
- new net GPIO22: J1.15 (Pin_15)
- new net GPIO23: J1.16 (Pin_16)
- new net GPIO24: J1.18 (Pin_18)
- new net GPIO25: J1.22 (Pin_22)
- new net GPIO26: J1.37 (Pin_37)
- new net GPIO27: J1.13 (Pin_13)
- new net GPIO2/SDA1: J1.3 (Pin_3)
- new net GPIO3/SCL1: J1.5 (Pin_5)
- new net GPIO4/GPCLK0: J1.7 (Pin_7)
- new net GPIO5: J1.29 (Pin_29)
- new net GPIO6: J1.31 (Pin_31)
- new net GPIO7/SPI0.CE1: J1.26 (Pin_26)
- new net GPIO8/SPI0.CE0: J1.24 (Pin_24), U1.20 (~{CS})
- new net GPIO9/SPI0.MISO: J1.21 (Pin_21), U1.22 (DOUT)
- new net ID_SCL: J1.28 (Pin_28)
- new net ID_SDA: J1.27 (Pin_27)
- no-connect marks 0 -> 4
Other:
- note added: "Additional pin functions: https://pinout.xyz/"

Commit message: bruh
Parts:
- added R1, R2, R3: 100, symbol Device:R
Connections:
- net GPIO10/SPI0.MOSI: now also R3.2; no longer U1.23 (DIN)
- net GPIO11/SPI0.SCLK: now also R2.2; no longer U1.24 (SCLK)
- net GPIO22: now also U1.21 (~{DRDY})
- net GPIO8/SPI0.CE0: now also R1.2; no longer U1.20 (~{CS})
- new net: R2.1, U1.24 (SCLK)
- new net: R1.1, U1.20 (~{CS})
- new net: R3.1, U1.23 (DIN)

Commit message: the
Parts:
- removed C2, C3, C4, C5, C6, C7: C, symbol Device:C
- removed R1, R2, R3: 100, symbol Device:R
- removed U1: ADS1256IDBR, 1Personal:IC_ADC_ADS1256IDBR, symbol Custom:ADS1256IDBR
- removed Y1: Crystal 8 MHz, symbol Device:Crystal
- added U1, U2: ADS1115IDGS, Package_SO:TSSOP-10_3x3mm_P0.5mm, symbol Analog_ADC:ADS1115IDGS
Connections:
- no-connect marks 4 -> 0
