File: Hardware/fatigue.kicad_sch (KiCad schematic)
At the start: 12 parts, among them J1 GPIO, U1 ADS1256IDBR, Y1 Crystal 8 MHz

Commit message: syncing this all up
Parts:
- removed C4, C5, C6, C7: C, symbol Device:C
- removed U1: ADS1256IDBR, 1Personal:IC_ADC_ADS1256IDBR, symbol Custom:ADS1256IDBR
- removed Y1: Crystal 8 MHz, symbol Device:Crystal
- added C1: 0.22 uF, symbol Device:C
- added R4, R5: 10k, symbol Device:R
- added U1, U2: ADS1115IDGS, Package_SO:TSSOP-10_3x3mm_P0.5mm, symbol Analog_ADC:ADS1115IDGS
- C2: footprint (none) -> 0.1 uF
- C3: value C -> 0.1 uF
- R1: value 100 -> R
- R2: value 100 -> 10k; footprint (none) -> Resistor_SMD:R_1206_3216Metric_Pad1.30x1.75mm_HandSolder
- R3: value 100 -> 10k
Connections:
- net +5V: now also C2.1, C3.1, R2.1, R3.1, R4.1, R5.1, U1.1 (ADDR), U1.8 (VDD), U2.8 (VDD); no longer J1.2 (Pin_2), J1.4 (Pin_4)
- net GND: now also C1.2, U1.3 (GND), U1.5 (AIN1), U1.6 (AIN2), U1.7 (AIN3), U2.1 (ADDR), U2.3 (GND), U2.5 (AIN1), U2.6 (AIN2), U2.7 (AIN3)
- net GPIO10/SPI0.MOSI: no longer R3.2
- net GPIO11/SPI0.SCLK: no longer R2.2
- net GPIO8/SPI0.CE0: no longer R1.2
- net LOADCELL_IN: now reaches R1.1
- new net: C1.1, R1.2, U1.4 (AIN0)
- new net: R2.2, U1.2 (ALERT/RDY)
- new net: R3.2, U1.10 (SCL), U2.10 (SCL)
- new net: R4.2, U1.9 (SDA), U2.9 (SDA)
- new net: R5.2, U2.2 (ALERT/RDY)
- new net LASER_IN: U2.4 (AIN0)
- new net PI +5V: J1.2 (Pin_2), J1.4 (Pin_4)
- no-connect marks 4 -> 0
