File: Hardware/modules/conditioner+adc module/ADC1.kicad_sch (KiCad schematic)
At the start: 8 parts, among them U4 ADS1115

Commit message: p
Connections:
- net AGND is gone; now on net GND: C10.2, C9.2, U4.3 (GND)
- net GND: now also U4.1 (ADDR)
