File: Hardware/modules/conditioner+adc module/ADC2.kicad_sch (KiCad schematic)
At the start: 8 parts, among them U4 ADS1115

Commit message: p
Parts:
- removed C10, C9: C, Capacitor_SMD:C_0805_2012Metric_Pad1.18x1.45mm_HandSolder, symbol Device:C
- removed C11: 0.1 uF, Capacitor_SMD:C_0805_2012Metric_Pad1.18x1.45mm_HandSolder, symbol Device:C
- removed D2: LED, LED_SMD:LED_0805_2012Metric_Pad1.15x1.40mm_HandSolder, symbol Device:LED
- removed R20, R21: R, Resistor_SMD:R_0805_2012Metric_Pad1.20x1.40mm_HandSolder, symbol Device:R
- removed R22: 1k, Resistor_SMD:R_0805_2012Metric_Pad1.20x1.40mm_HandSolder, symbol Device:R
- removed U4: ADS1115, Package_SO:TSSOP-10_3x3mm_P0.5mm, symbol Analog_ADC:ADS1115IDGS
- added C3, C4: C, Capacitor_SMD:C_0805_2012Metric_Pad1.18x1.45mm_HandSolder, symbol Device:C
- added C5: 0.1 uF, Capacitor_SMD:C_0805_2012Metric_Pad1.18x1.45mm_HandSolder, symbol Device:C
- added D1: LED, LED_SMD:LED_0805_2012Metric_Pad1.15x1.40mm_HandSolder, symbol Device:LED
- added R11, R12: R, Resistor_SMD:R_0805_2012Metric_Pad1.20x1.40mm_HandSolder, symbol Device:R
- added R13: 1k, Resistor_SMD:R_0805_2012Metric_Pad1.20x1.40mm_HandSolder, symbol Device:R
- added U2: ADS1115, Package_SO:TSSOP-10_3x3mm_P0.5mm, symbol Analog_ADC:ADS1115IDGS
Connections:
- net +5V: now also C5.2, D1.2 (A), U2.1 (ADDR), U2.8 (VDD)
- net AGND: now also C3.2, C4.2, U2.3 (GND)
- net GND: now also C5.1, R13.2
- net Input: now also R11.1
- net SCL: now also U2.10 (SCL)
- net SDA: now also U2.9 (SDA)
- new net: C4.1, R12.2, U2.5 (AIN1)
- new net: C3.1, R11.2, U2.4 (AIN0)
- new net: D1.1 (K), R13.1

Commit message: p
Connections:
- net AGND is gone; now on net GND: C3.2, C4.2, U2.3 (GND)
Changed lines of the file:
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@@
 	)
 	(symbol
-		(lib_id "power:GNDA")
+		(lib_id "power:GND")
 		(at 128.27 109.22 0)
 		(unit 1)
@@
 			)
 		)
-		(property "Value" "AGND"
+		(property "Value" "GND"
 			(at 128.27 114.3 0)
 			(effects
@@
 			)
 		)
-		(property "Description" "Power symbol creates a global label with name \"GNDA\" , analog ground"
+		(property "Description" "Power symbol creates a global label with name \"GND\" , ground"
 			(at 128.27 109.22 0)
 			(effects
