File: Hardware/modules/conditioner+adc module/Conditioner1.kicad_sch (KiCad schematic)
At the start: 20 parts, among them P1-5k1 TRIM_TS63Y, P2-5k1 TRIM_TS63Y

Commit message: up
Parts:
- removed P1-5k1, P2-5k1: TRIM_TS63Y, 1Personal:TRIM_TS63Y, symbol Custom:TRIM_TS63Y
- removed R11: 130, Resistor_SMD:R_0603_1608Metric_Pad0.98x0.95mm_HandSolder, symbol Device:R
- removed R12: 1.58, Resistor_SMD:R_0603_1608Metric_Pad0.98x0.95mm_HandSolder, symbol Device:R
- removed R5: 33.2, Resistor_SMD:R_0805_2012Metric_Pad1.20x1.40mm_HandSolder, symbol Device:R
- R10: value 2.5K -> 3160; footprint Resistor_SMD:R_0603_1608Metric_Pad0.98x0.95mm_HandSolder -> Resistor_SMD:R_1206_3216Metric_Pad1.30x1.75mm_HandSolder
- R3: value 10k -> 10.2k; footprint Resistor_SMD:R_0805_2012Metric_Pad1.20x1.40mm_HandSolder -> Resistor_SMD:R_1206_3216Metric_Pad1.30x1.75mm_HandSolder
- R4: value 3.3k -> 3400; footprint Resistor_SMD:R_0805_2012Metric_Pad1.20x1.40mm_HandSolder -> Resistor_SMD:R_1206_3216Metric_Pad1.30x1.75mm_HandSolder
- R9: value 10k -> 12k; footprint Resistor_SMD:R_0805_2012Metric_Pad1.20x1.40mm_HandSolder -> Resistor_SMD:R_1206_3216Metric_Pad1.30x1.75mm_HandSolder
Connections:
- net AGND: now also R10.2, R4.1
- net at R3.1, TP1.1, U1.5 (+In_B): now also R4.2; no longer R4.1
- no-connect marks 2 -> 0

Commit message: p
Parts:
- removed R13, R8: 10k, Resistor_SMD:R_0805_2012Metric_Pad1.20x1.40mm_HandSolder, symbol Device:R
- added R10, R5: 10k, Resistor_SMD:R_0805_2012Metric_Pad1.20x1.40mm_HandSolder, symbol Device:R
- renumbered R9 to R8, R10 to R9
Connections:
- net +In_D: now also R6.2, R5.1; no longer R6.1, R7.2
- net AGND: now also R10.2
- net Output: now also R7.1
- net at U1.13 (-In_D): now also R7.2, R10.1
- net +2.5V: now reaches R8.1, R9.1, TP2.1, U1.10 (+In_C)
- net at U1.8 (Out_C), U1.9 (-In_C): now also R6.1; no longer R7.1
- net at U1.6 (-In_B), U1.7 (Out_B): now also R5.2; no longer R6.2

Commit message: p
Connections:
- net +2.5V: no longer names the net of R8.1, R9.1, TP2.1, U1.10 (+In_C)
- net AGND renamed GND
