File: Hardware/modules/conditioner+adc module/Conditioner2.kicad_sch (KiCad schematic)
At the start: 11 parts

Commit message: p
Parts:
- removed C7, C8: 0.1 uF, Capacitor_SMD:C_0805_2012Metric_Pad1.18x1.45mm_HandSolder, symbol Device:C
- added C12: 0.1 uF, Capacitor_SMD:C_0805_2012Metric_Pad1.18x1.45mm_HandSolder, symbol Device:C
- added R25, R26: 10k, Resistor_SMD:R_1206_3216Metric_Pad1.30x1.75mm_HandSolder, symbol Device:R
- added R27: 12k, Resistor_SMD:R_1206_3216Metric_Pad1.30x1.75mm_HandSolder, symbol Device:R
- added R28: 3160, Resistor_SMD:R_1206_3216Metric_Pad1.30x1.75mm_HandSolder, symbol Device:R
Connections:
- net AGND is gone; now on net GND: C6.2, R15.1, R19.2
- net +12V: now also R25.2, R27.1
- net -12V: now also C12.2, R26.2
- net GND: now reaches U3.1 (Out_A)
- net GND: now also U3.2 (-In_A), C12.1, R28.2
- net at U3.3 (+In_A): now also R25.1, R26.1
- net +2.5V: no longer names the net of U3.10 (+In_C)
- net +2.5V: now also R27.2, R28.1
- no-connect marks 3 -> 0
Other:
- moved on the sheet: C6
