File: Hardware/modules/conditioner+adc module/conditioner+adc.kicad_pcb (KiCad board)
At the start: 2 copper layers, 26.7 x 22.2 mm, 19 parts, among them J1 Conn_01x08_MountingPin, J2 Conn_01x08_MountingPin

Commit message: updates
Parts:
- removed J1, J2: Conn_01x08_MountingPin, Connector_PinHeader_2.54mm:PinHeader_1x08_P2.54mm_Vertical
- removed R9: 1k, Resistor_SMD:R_0805_2012Metric_Pad1.20x1.40mm_HandSolder
- added C3: 0.1 uF, Capacitor_SMD:C_0805_2012Metric_Pad1.18x1.45mm_HandSolder, F.Cu at (138.7, 75.9)
- added C4: 0.1 uF, Capacitor_SMD:C_0805_2012Metric_Pad1.18x1.45mm_HandSolder, F.Cu at (198.8, 130.8)
- added C4_OPT1: C, Capacitor_SMD:C_0805_2012Metric_Pad1.18x1.45mm_HandSolder, F.Cu at (137.3, 84.7)
- added C4_OPT2: C, Capacitor_SMD:C_0805_2012Metric_Pad1.18x1.45mm_HandSolder, F.Cu at (198.8, 133.8)
- added C5_OPT1: C, Capacitor_SMD:C_0805_2012Metric_Pad1.18x1.45mm_HandSolder, F.Cu at (140.5, 86.0)
- added C5_OPT2: C, Capacitor_SMD:C_0805_2012Metric_Pad1.18x1.45mm_HandSolder, F.Cu at (204.1, 90.6)
- added D1: LED, LED_SMD:LED_0805_2012Metric_Pad1.15x1.40mm_HandSolder, F.Cu at (142.2, 77.0)
- added D2: LED, LED_SMD:LED_0805_2012Metric_Pad1.15x1.40mm_HandSolder, F.Cu at (184.0, 95.5)
- added J3: Conn_02x20_RaspberryPi_40Pin, 1Personal:CONN_RASPBERRYPI_40PIN_2x20, F.Cu at (128.5, 66.2)
- added P1-5k1: TRIM_TS63Y, 1Personal:TRIM_TS63Y, F.Cu at (145.7, 101.5)
- added P2-5k1: TRIM_TS63Y, 1Personal:TRIM_TS63Y, F.Cu at (130.1, 99.8)
- added R15: 1k, Resistor_SMD:R_0805_2012Metric_Pad1.20x1.40mm_HandSolder, F.Cu at (141.6, 75.0)
- added R17: 1k, Resistor_SMD:R_0805_2012Metric_Pad1.20x1.40mm_HandSolder, F.Cu at (134.7, 73.8)
- added R18: 1k, Resistor_SMD:R_0805_2012Metric_Pad1.20x1.40mm_HandSolder, F.Cu at (135.7, 76.0)
- added R19: R, Resistor_SMD:R_0805_2012Metric_Pad1.20x1.40mm_HandSolder, F.Cu at (194.0, 130.8)
- added R19_OPT1: R, Resistor_SMD:R_0805_2012Metric_Pad1.20x1.40mm_HandSolder, F.Cu at (138.3, 87.6)
- added R19_OPT2: R, Resistor_SMD:R_0805_2012Metric_Pad1.20x1.40mm_HandSolder, F.Cu at (199.3, 96.4)
- added R20: 1k, Resistor_SMD:R_0805_2012Metric_Pad1.20x1.40mm_HandSolder, F.Cu at (194.0, 133.7)
- added R20_OPT1: R, Resistor_SMD:R_0805_2012Metric_Pad1.20x1.40mm_HandSolder, F.Cu at (141.6, 83.1)
- added R20_OPT2: R, Resistor_SMD:R_0805_2012Metric_Pad1.20x1.40mm_HandSolder, F.Cu at (199.3, 99.3)
- added R21: 1k, Resistor_SMD:R_0805_2012Metric_Pad1.20x1.40mm_HandSolder, F.Cu at (199.3, 90.5)
- added R22: 1k, Resistor_SMD:R_0805_2012Metric_Pad1.20x1.40mm_HandSolder, F.Cu at (199.3, 93.4)
- added TP1: TestPoint, TestPoint:TestPoint_Pad_D2.0mm, F.Cu at (124.6, 100.5)
- added TP2: TestPoint, TestPoint:TestPoint_Pad_D2.0mm, F.Cu at (148.2, 96.0)
- added U2: ADS1115, Package_SO:TSSOP-10_3x3mm_P0.5mm, F.Cu at (137.8, 80.8)
- added U3: ADS1115, Package_SO:TSSOP-10_3x3mm_P0.5mm, F.Cu at (179.4, 102.7)
- R4: footprint Resistor_SMD:R_1206_3216Metric_Pad1.30x1.75mm_HandSolder -> Resistor_SMD:R_0603_1608Metric_Pad0.98x0.95mm_HandSolder
- moved R1 46.5 mm to (128.7, 99.7), turned to -90 degrees
- moved R4 46.3 mm to (142.7, 101.5), turned to -90 degrees
- moved R2 46.2 mm to (127.8, 94.2), turned to 90 degrees
- moved R13 43.9 mm to (142.7, 90.6), turned to -90 degrees
- moved R10 43.7 mm to (143.6, 96.8)
- moved C2 43.7 mm to (143.6, 94.8)
- moved U1 43.7 mm to (137.9, 94.7)
- moved R12 43.6 mm to (139.8, 100.3), turned to 180 degrees
- moved R5 43.5 mm to (145.4, 101.6), turned to 90 degrees
- moved C1 43.5 mm to (132.3, 94.8)
- moved R3 43.1 mm to (131.6, 101.8), turned to 0 degrees
- moved R11 42.7 mm to (136.1, 100.3), turned to 180 degrees
- moved R7 42.4 mm to (133.3, 91.8), turned to 90 degrees
- moved R14 41.6 mm to (144.8, 90.6), turned to 90 degrees
- moved R8 40.5 mm to (134.3, 88.9), turned to 0 degrees
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Connections:
- net /output renamed /Cond1Output
- C1 pad 2: GND -> AGND
- C2 pad 1: GND -> AGND
- R14 pad 2: GND -> AGND
- R3 pad 2: GND -> AGND
- R6 pad 2: GND -> AGND
- U1 pad 1: Net-(U1-Out_A) -> AGND
- U1 pad 2: GND -> AGND
Routing:
- net +12V: track 36.8 -> 5.62 mm, vias 0 -> 1
- net /+In_D: track 30.0 -> 10.2 mm
- net AGND: track 0.00 -> 19.1 mm, vias 0 -> 7
- net -12V: track 25.4 -> 6.48 mm, vias 0 -> 2
- net /SCL: track 0.00 -> 18.6 mm
- net /SDA: track 0.00 -> 13.1 mm
- net Net-(U1-+In_B): track 4.98 -> 16.5 mm
- net /LC_S: track 11.1 -> 0.00 mm
- net +5V: track 0.00 -> 9.46 mm, vias 0 -> 1
- net Net-(U1-+In_C): track 4.51 -> 12.9 mm
- net Net-(U2-AIN0): track 0.00 -> 3.74 mm
- net Net-(U2-AIN1): track 0.00 -> 3.64 mm
- net Net-(U1-+In_A): track 6.50 -> 2.92 mm
- net GND: track 0.00 -> 3.48 mm, vias 17 -> 1
- net Net-(U1--In_B): track 0.00 -> 3.23 mm
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- added copper zone on In1.Cu, net AGND
- added copper zone on In1.Cu, net GND
- removed copper zone on F.Cu, net /Cond1Output
- removed copper zone on B.Cu, net GND
- removed copper zone on F.Cu, net GND
- removed copper zone on F.Cu, net Net-(U1--In_B)
- removed copper zone on F.Cu, net Net-(U1--In_C)
Other:
- board size 26.7 x 22.2 mm -> 108.4 x 62.1 mm
- copper layers 2 -> 4
- board text removed: "+12V"
- board text removed: "-12V"
- board text removed: "GND"
- board text removed: "LC"
- board text removed: "Signal Conditioner Module"
- board text removed: "Tyler Patterson - Rev 1"
- board text removed: "Vout"

Commit message: p
Parts:
- removed C4_OPT1, C4_OPT2, C5_OPT2: C, Capacitor_SMD:C_0805_2012Metric_Pad1.18x1.45mm_HandSolder
- removed J3: Conn_02x20_RaspberryPi_40Pin, 1Personal:CONN_RASPBERRYPI_40PIN_2x20
- removed R17, R18, R22: 1k, Resistor_SMD:R_0805_2012Metric_Pad1.20x1.40mm_HandSolder
- removed R19_OPT1, R19_OPT2, R20_OPT1, R20_OPT2: R, Resistor_SMD:R_0805_2012Metric_Pad1.20x1.40mm_HandSolder
- added C10: 0.1 uF, Capacitor_SMD:C_0805_2012Metric_Pad1.18x1.45mm_HandSolder, F.Cu at (149.0, 71.8)
- added C6: C, Capacitor_SMD:C_0805_2012Metric_Pad1.18x1.45mm_HandSolder, F.Cu at (147.9, 80.7)
- added C7: C, Capacitor_SMD:C_0805_2012Metric_Pad1.18x1.45mm_HandSolder, F.Cu at (151.1, 78.0)
- added C8: 0.1 uF, Capacitor_SMD:C_0805_2012Metric_Pad1.18x1.45mm_HandSolder, F.Cu at (156.1, 88.9)
- added C9: 0.1 uF, Capacitor_SMD:C_0805_2012Metric_Pad1.18x1.45mm_HandSolder, F.Cu at (167.3, 88.9)
- added J1: Conn_02x20_RaspberryPi_40Pin, 1Personal:CONN_RASPBERRYPI_40PIN_2x20, F.Cu at (120.7, 65.3)
- added J2: CONN_JST_1x2_1.25mmPitch, 1Personal:CONN_JST_1x2_1.25mmPitch, F.Cu at (111.3, 69.5)
- added P1-5k5: TRIM_TS63Y, 1Personal:TRIM_TS63Y, F.Cu at (112.5, 81.8)
- added P3-5k1: TRIM_TS63Y, 1Personal:TRIM_TS63Y, F.Cu at (153.2, 95.0)
- added P4-5k1: TRIM_TS63Y, 1Personal:TRIM_TS63Y, F.Cu at (169.5, 95.6)
- added R16: 1k, Resistor_SMD:R_0805_2012Metric_Pad1.20x1.40mm_HandSolder, F.Cu at (132.7, 74.0)
- added R32: 10k, Resistor_SMD:R_0805_2012Metric_Pad1.20x1.40mm_HandSolder, F.Cu at (155.2, 86.9)
- added R33: 10k, Resistor_SMD:R_0805_2012Metric_Pad1.20x1.40mm_HandSolder, F.Cu at (155.2, 84.8)
- added R34: 10k, Resistor_SMD:R_0805_2012Metric_Pad1.20x1.40mm_HandSolder, F.Cu at (150.5, 88.8)
- added R35: 3.3k, Resistor_SMD:R_0805_2012Metric_Pad1.20x1.40mm_HandSolder, F.Cu at (151.8, 93.5)
- added R36: 33.2, Resistor_SMD:R_0805_2012Metric_Pad1.20x1.40mm_HandSolder, F.Cu at (154.6, 93.8)
- added R37: 10k, Resistor_SMD:R_0805_2012Metric_Pad1.20x1.40mm_HandSolder, F.Cu at (159.8, 94.6)
- added R38: 10k, Resistor_SMD:R_0805_2012Metric_Pad1.20x1.40mm_HandSolder, F.Cu at (163.5, 94.6)
- added R39: 10k, Resistor_SMD:R_0805_2012Metric_Pad1.20x1.40mm_HandSolder, F.Cu at (167.4, 84.3)
- added R40: 10k, Resistor_SMD:R_0805_2012Metric_Pad1.20x1.40mm_HandSolder, F.Cu at (163.6, 97.8)
- added R41: 2.5K, Resistor_SMD:R_0603_1608Metric_Pad0.98x0.95mm_HandSolder, F.Cu at (167.8, 94.2)
- added R42: 130, Resistor_SMD:R_0603_1608Metric_Pad0.98x0.95mm_HandSolder, F.Cu at (169.5, 96.2)
- added R43: 1.58, Resistor_SMD:R_0603_1608Metric_Pad0.98x0.95mm_HandSolder, F.Cu at (171.1, 96.7)
- added R44: 10k, Resistor_SMD:R_0805_2012Metric_Pad1.20x1.40mm_HandSolder, F.Cu at (167.5, 86.4)
- added R9: 10k, Resistor_SMD:R_0805_2012Metric_Pad1.20x1.40mm_HandSolder, F.Cu at (133.6, 97.7)
- added TP5: TestPoint, TestPoint:TestPoint_Pad_D2.0mm, F.Cu at (159.1, 99.9)
- added TP6: TestPoint, TestPoint:TestPoint_Pad_D2.0mm, F.Cu at (173.6, 89.9)
- added U4: ~, Package_SO:SOIC-14_3.9x8.7mm_P1.27mm, F.Cu at (161.7, 88.8)
- added U5: IC_LinearRegulator_1-30VOutput, 1Personal:IC_LinearRegulator_1-30VOutput, F.Cu at (119.6, 75.6)
- C3, C4: value 0.1 uF -> C
- C5: renamed from C5_OPT1; value C -> 0.1 uF
- R1: value 3.3k -> 10k
- R10: value 10k -> 2.5K; footprint Resistor_SMD:R_0805_2012Metric_Pad1.20x1.40mm_HandSolder -> Resistor_SMD:R_0603_1608Metric_Pad0.98x0.95mm_HandSolder
- R11: value 10k -> 130; footprint Resistor_SMD:R_0805_2012Metric_Pad1.20x1.40mm_HandSolder -> Resistor_SMD:R_0603_1608Metric_Pad0.98x0.95mm_HandSolder
- R12: value 10k -> 1.58; footprint Resistor_SMD:R_0805_2012Metric_Pad1.20x1.40mm_HandSolder -> Resistor_SMD:R_0603_1608Metric_Pad0.98x0.95mm_HandSolder
- R14: value 10k -> R
- R15, R20: value 1k -> R
- R3: value 33.2 -> 10k
- R4: value 2.5K -> 3.3k; footprint Resistor_SMD:R_0603_1608Metric_Pad0.98x0.95mm_HandSolder -> Resistor_SMD:R_0805_2012Metric_Pad1.20x1.40mm_HandSolder
- R5: value 130 -> 33.2; footprint Resistor_SMD:R_0603_1608Metric_Pad0.98x0.95mm_HandSolder -> Resistor_SMD:R_0805_2012Metric_Pad1.20x1.40mm_HandSolder
- R6: value 1.58 -> 10k; footprint Resistor_SMD:R_0603_1608Metric_Pad0.98x0.95mm_HandSolder -> Resistor_SMD:R_0805_2012Metric_Pad1.20x1.40mm_HandSolder
- moved C4 84.7 mm to (132.6, 78.0)
- moved R19 69.5 mm to (145.9, 80.7), turned to 90 degrees
- moved R20 68.8 mm to (151.1, 80.0), turned to 180 degrees
- moved R21 50.9 mm to (151.2, 74.0), turned to 180 degrees
- moved U3 41.9 mm to (147.4, 75.7)
- moved D2 36.1 mm to (155.0, 74.0)
- moved R4 22.3 mm to (121.8, 93.4)
- moved R5 22.2 mm to (124.6, 93.7), turned to -90 degrees
- moved R14 20.1 mm to (127.4, 80.7)
- moved R6 17.7 mm to (129.8, 94.4), turned to 180 degrees
- moved C5 17.3 mm to (130.5, 71.8), turned to 180 degrees
- moved R3 17.2 mm to (120.5, 88.7), turned to 180 degrees
- moved R1 13.4 mm to (125.2, 86.8), turned to 180 degrees
- moved C3 10.4 mm to (129.4, 80.7)
- moved R15 10.3 mm to (132.5, 80.0)
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- renumbered P2-5k1 to P1-5k1, P1-5k1 to P2-5k1
Connections:
- C3 pad 1: GND -> Net-(U2-AIN0)
- C3 pad 2: +5V -> AGND
- C4 pad 1: Net-(C4-Pad1) -> Net-(U2-AIN1)
- C4 pad 2: +5V -> AGND
- C5 pad 1: Net-(U2-AIN1) -> GND
- C5 pad 2: AGND -> +5V
- R1 pad 1: Net-(U1-+In_B) -> +12V
- R1 pad 2: Net-(R1-Pad2) -> Net-(U1-+In_A)
- R10 pad 2: +12V -> Net-(R10-Pad2)
- R11 pad 1: /+In_D -> Net-(R10-Pad2)
- R11 pad 2: Net-(U1--In_B) -> Net-(R11-Pad2)
- R12 pad 1: Net-(U1--In_C) -> Net-(R11-Pad2)
- R12 pad 2: /+In_D -> AGND
- R13 pad 1: /Cond1Output -> Net-(U1--In_D)
- R13 pad 2: Net-(U1--In_D) -> AGND
- R14 pad 1: Net-(U1--In_D) -> /ADC1/Input
- R14 pad 2: AGND -> Net-(U2-AIN0)
- R15 pad 1: Net-(D1-K) -> unconnected-(R15-Pad1)
- R15 pad 2: GND -> Net-(U2-AIN1)
- R19 pad 1: Net-(D2-K) -> /ADC2/Input
- R19 pad 2: Net-(C4-Pad1) -> Net-(U3-AIN0)
- R2 pad 1: Net-(U1-+In_B) -> Net-(U1-+In_A)
- R2 pad 2: /LC_S -> -12V
- R20 pad 1: +5V -> unconnected-(R20-Pad1)
- R20 pad 2: Net-(U3-ADDR) -> Net-(U3-AIN1)
- R21 pad 1: +5V -> Net-(D2-K)
- R21 pad 2: Net-(U3-SDA) -> GND
- R3 pad 1: Net-(R1-Pad2) -> Net-(U1-+In_B)
- R3 pad 2: AGND -> /Conditioner1/Input
- R4 pad 1: Net-(U1-+In_C) -> Net-(U1-+In_B)
- R5 pad 2: Net-(R5-Pad2) -> AGND
- R6 pad 1: Net-(R5-Pad2) -> /Conditioner1/+In_D
- R6 pad 2: AGND -> Net-(U1--In_B)
- R7 pad 1: +12V -> Net-(U1--In_C)
- R7 pad 2: Net-(U1-+In_A) -> /Conditioner1/+In_D
- R8 pad 1: Net-(U1-+In_A) -> /Conditioner1/Output
- R8 pad 2: -12V -> Net-(U1--In_D)
- U1 pad 12: /+In_D -> /Conditioner1/+In_D
- U1 pad 14: /Cond1Output -> /Conditioner1/Output
- U2 pad 1: AGND -> /ADC1/SCL
- U2 pad 10: /SCL -> /ADC1/SCL
- U2 pad 9: /SDA -> /ADC1/SDA
- U3 pad 1: Net-(U3-ADDR) -> /ADC1/SCL
- U3 pad 10: Net-(U3-ADDR) -> /ADC1/SCL
- U3 pad 2: Net-(U3-ALRT) -> unconnected-(U3-ALRT-Pad2)
- U3 pad 9: Net-(U3-SDA) -> /ADC1/SDA
Routing:
- net +5V: track 9.46 -> 55.6 mm, vias 1 -> 0
- net Net-(U4-+In_B): track 0.00 -> 21.6 mm
- net Net-(U4-+In_C): track 0.00 -> 19.1 mm
- net AGND: track 19.1 -> 32.0 mm, vias 7 -> 16
- net /SCL: track 18.6 -> 6.89 mm
- net /Conditioner1/Output: track 0.00 -> 11.3 mm
- net /+In_D: track 10.2 -> 0.00 mm
- net /Conditioner2/+In_D: track 0.00 -> 10.1 mm
- net /Conditioner1/+In_D: track 0.00 -> 10.1 mm
- net Net-(U4-+In_A): track 0.00 -> 8.62 mm
- net Net-(U1-+In_C): track 12.9 -> 19.1 mm
- net +12V: track 5.62 -> 11.8 mm, vias 1 -> 2
- net /Cond1Output: track 5.92 -> 0.00 mm
- net Net-(U1-+In_A): track 2.92 -> 8.62 mm
- net Net-(U4--In_D): track 0.00 -> 5.44 mm
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Other:
- board size 108.4 x 62.1 mm -> 70.9 x 39.7 mm

Commit message: up
Parts:
- removed P1-5k1, P2-5k1, P3-5k1, P4-5k1: TRIM_TS63Y, 1Personal:TRIM_TS63Y
- removed R11, R42: 130, Resistor_SMD:R_0603_1608Metric_Pad0.98x0.95mm_HandSolder
- removed R12, R43: 1.58, Resistor_SMD:R_0603_1608Metric_Pad0.98x0.95mm_HandSolder
- removed R35: 3.3k, Resistor_SMD:R_0805_2012Metric_Pad1.20x1.40mm_HandSolder
- removed R36: 33.2, Resistor_SMD:R_0805_2012Metric_Pad1.20x1.40mm_HandSolder
- added R17: 10k, Resistor_SMD:R_0805_2012Metric_Pad1.20x1.40mm_HandSolder, F.Cu at (155.3, 108.2)
- added R18: 10k, Resistor_SMD:R_0805_2012Metric_Pad1.20x1.40mm_HandSolder, F.Cu at (150.0, 111.0)
- R10, R41: value 2.5K -> 3160; footprint Resistor_SMD:R_0603_1608Metric_Pad0.98x0.95mm_HandSolder -> Resistor_SMD:R_1206_3216Metric_Pad1.30x1.75mm_HandSolder
- R3, R34: value 10k -> 10.2k; footprint Resistor_SMD:R_0805_2012Metric_Pad1.20x1.40mm_HandSolder -> Resistor_SMD:R_1206_3216Metric_Pad1.30x1.75mm_HandSolder
- R4: value 3.3k -> 3400; footprint Resistor_SMD:R_0805_2012Metric_Pad1.20x1.40mm_HandSolder -> Resistor_SMD:R_1206_3216Metric_Pad1.30x1.75mm_HandSolder
- R40, R9: value 10k -> 12k; footprint Resistor_SMD:R_0805_2012Metric_Pad1.20x1.40mm_HandSolder -> Resistor_SMD:R_1206_3216Metric_Pad1.30x1.75mm_HandSolder
- R5: value 33.2 -> 3400; footprint Resistor_SMD:R_0805_2012Metric_Pad1.20x1.40mm_HandSolder -> Resistor_SMD:R_1206_3216Metric_Pad1.30x1.75mm_HandSolder
- moved R5 27.1 mm to (151.7, 94.4), turned to 90 degrees
- moved R3 0.25 mm to (120.2, 88.7)
- moved R4 0.20 mm to (121.7, 93.5), turned to 90 degrees
Connections:
- P1-5k5 pad 2: unconnected-(P1-5k5-Pad2) -> Net-(U5-FB)
- R10 pad 2: Net-(R10-Pad2) -> AGND
- R4 pad 1: Net-(U1-+In_B) -> AGND
- R4 pad 2: Net-(R4-Pad2) -> Net-(U1-+In_B)
- R41 pad 2: Net-(R41-Pad2) -> AGND
- R5 pad 1: Net-(R4-Pad2) -> AGND
- R5 pad 2: AGND -> Net-(U4-+In_B)
Routing:
- net Net-(R35-Pad2): track 3.47 -> 0.00 mm
- net Net-(R4-Pad2): track 3.47 -> 0.00 mm
- net Net-(R42-Pad2): track 1.81 -> 0.00 mm
- net Net-(R11-Pad2): track 1.81 -> 0.00 mm
- net Net-(R10-Pad2): track 1.76 -> 0.00 mm
- net Net-(R41-Pad2): track 1.76 -> 0.00 mm
- net AGND: track 32.0 -> 33.6 mm

Commit message: p
Parts:
- removed the C9 at (167.3, 88.9)
- removed P1-5k5: TRIM_TS63Y, 1Personal:TRIM_TS63Y
- removed the R17 at (155.3, 108.2)
- removed the R18 at (150.0, 111.0)
- removed R32, R33: 10k, Resistor_SMD:R_0805_2012Metric_Pad1.20x1.40mm_HandSolder
- removed R40: 12k, Resistor_SMD:R_1206_3216Metric_Pad1.30x1.75mm_HandSolder
- removed R41: 3160, Resistor_SMD:R_1206_3216Metric_Pad1.30x1.75mm_HandSolder
- removed TP6: TestPoint, TestPoint:TestPoint_Pad_D2.0mm
- removed U5: IC_LinearRegulator_1-30VOutput, 1Personal:IC_LinearRegulator_1-30VOutput
- added C6: 0.1 uF, Capacitor_SMD:C_0805_2012Metric_Pad1.18x1.45mm_HandSolder, F.Cu at (157.0, 87.0)
- added C7: 0.1 uF, Capacitor_SMD:C_0805_2012Metric_Pad1.18x1.45mm_HandSolder, F.Cu at (167.3, 91.1)
- added J1: CONN_JST_1x2_1.25mmPitch, 1Personal:CONN_JST_1x2_1.25mmPitch, F.Cu at (111.0, 69.3)
- added J3: CONN_JST_1x2_1.25mmPitch, 1Personal:CONN_JST_1x2_1.25mmPitch, F.Cu at (125.8, 100.5)
- moved J2 52.6 mm to (153.7, 100.6), turned to 0 degrees
- moved TP1 14.1 mm to (119.2, 89.8)
- moved C8 11.3 mm to (167.4, 89.2), turned to 0 degrees
- moved R15 8.48 mm to (154.7, 86.5), turned to -90 degrees
- moved R3 7.95 mm to (126.5, 93.7), turned to -90 degrees
- moved R14 4.11 mm to (153.5, 91.6), turned to -90 degrees
- moved TP2 3.50 mm to (141.9, 92.8)
- renumbered C4 to C10, C5 to C11, C6 to C3, C7 to C4, C10 to C5, C3 to C9, D2 to D1, D1 to D2, J1 to J4, R13 to R10, R19 to R11, R20 to R12, R21 to R13, R34 to R14, R5 to R15, R37 to R16, R38 to R17, R39 to R18, R44 to R19, R14 to R20, R15 to R21, R16 to R22, R6 to R5, R7 to R6, R8 to R7, R9 to R8, R10 to R9, TP5 to TP3, U3 to U2, U4 to U3, U2 to U4
Connections:
- C8 pad 1: +12V -> -12V
- J2 pad 1: Net-(U5-EN) -> AGND
- J2 pad 2: GND -> /Conditioner2/Input
- R8 pad 1: Net-(U1-+In_C) -> /Conditioner1/+2.5V
- R9 pad 1: Net-(U1-+In_C) -> /Conditioner1/+2.5V
- TP2 pad 1: Net-(U1-+In_C) -> /Conditioner1/+2.5V
- U1 pad 10: Net-(U1-+In_C) -> /Conditioner1/+2.5V
- U2 pad 1: /ADC1/SCL -> +5V
- U3 pad 1: AGND -> unconnected-(U3-Out_A-Pad1)
- U3 pad 10: Net-(U4-+In_C) -> /Conditioner1/+2.5V
- U3 pad 2: AGND -> unconnected-(U3--In_A-Pad2)
- U3 pad 3: Net-(U4-+In_A) -> unconnected-(U3-+In_A-Pad3)
- U4 pad 1: /ADC1/SCL -> unconnected-(U4-ADDR-Pad1)
Routing:
- net /Conditioner1/+2.5V: track 0.00 -> 21.0 mm
- net Net-(U1-+In_C): track 18.9 -> 0.00 mm
- net Net-(U4-+In_C): track 18.9 -> 0.00 mm
- net Net-(U4-+In_A): track 8.62 -> 0.00 mm
- net Net-(U1-+In_B): track 21.6 -> 14.5 mm
- net /Conditioner2/Input: track 0.00 -> 5.27 mm
- net AGND: track 33.6 -> 38.0 mm, vias 16 -> 15
- net +5V: track 55.6 -> 58.6 mm
- net /Conditioner1/Input: track 0.00 -> 3.01 mm
- net +12V: track 11.8 -> 14.6 mm, vias 2 -> 3
- net -12V: track 11.7 -> 9.78 mm, vias 4 -> 3
- net Net-(U3-+In_B): track 21.6 -> 22.4 mm
Other:
- board size 70.9 x 39.7 mm -> 70.9 x 39.9 mm

Commit message: p
Parts:
- removed C7, C8: 0.1 uF, Capacitor_SMD:C_0805_2012Metric_Pad1.18x1.45mm_HandSolder
- added C12: 0.1 uF, Capacitor_SMD:C_0805_2012Metric_Pad1.18x1.45mm_HandSolder, F.Cu at (167.7, 89.1)
- added J5: Conn_01x06, 1Personal:CONN_JST_1x6_1.25mmPitch, F.Cu at (139.8, 60.0)
- added J6: Conn_01x03, 1Personal:CONN_JST_1x3_1.25mmPitch, F.Cu at (129.6, 60.0)
- added R23: 10k, Resistor_SMD:R_0805_2012Metric_Pad1.20x1.40mm_HandSolder, F.Cu at (145.2, 71.8)
- added R24: 10k, Resistor_SMD:R_0805_2012Metric_Pad1.20x1.40mm_HandSolder, F.Cu at (138.6, 71.7)
- added R25: 10k, Resistor_SMD:R_1206_3216Metric_Pad1.30x1.75mm_HandSolder, F.Cu at (154.4, 85.5)
- added R26: 10k, Resistor_SMD:R_1206_3216Metric_Pad1.30x1.75mm_HandSolder, F.Cu at (154.4, 83.2)
- added R27: 12k, Resistor_SMD:R_1206_3216Metric_Pad1.30x1.75mm_HandSolder, F.Cu at (166.3, 98.1)
- added R28: 3160, Resistor_SMD:R_1206_3216Metric_Pad1.30x1.75mm_HandSolder, F.Cu at (168.4, 93.1)
- moved J1 8.21 mm to (118.2, 73.2)
- moved R15 5.50 mm to (156.2, 91.8), turned to 90 degrees
- moved C6 1.39 mm to (156.1, 88.1), turned to 180 degrees
Connections:
- C1 pad 2: AGND -> GND
- C10 pad 2: AGND -> GND
- C2 pad 1: AGND -> GND
- C3 pad 2: AGND -> GND
- C4 pad 2: AGND -> GND
- C6 pad 2: AGND -> GND
- C9 pad 2: AGND -> GND
- J1 pad 1: unconnected-(J1-Pad1) -> +12V
- J1 pad 2: unconnected-(J1-Pad2) -> -12V
- J2 pad 1: AGND -> GND
- J3 pad 1: AGND -> GND
- J4 pad 2: /SDA -> /ADC1/SDA
- J4 pad 3: /SCL -> /ADC1/SCL
- J4 pad 33: unconnected-(J4-Pin_33-Pad33) -> /GPIO 23
- J4 pad 36: unconnected-(J4-Pin_36-Pad36) -> /UART RX
- J4 pad 37: unconnected-(J4-Pin_37-Pad37) -> /UART TX
- J4 pad 6: unconnected-(J4-Pin_6-Pad6) -> /GPIO 17
- J4 pad 7: unconnected-(J4-Pin_7-Pad7) -> /GPIO 27
- J4 pad 8: unconnected-(J4-Pin_8-Pad8) -> /GPIO 22
- R10 pad 2: AGND -> GND
- R15 pad 1: AGND -> GND
- R18 pad 1: /Conditioner2/Output -> /ADC2/Input
- R19 pad 2: AGND -> GND
- R4 pad 1: AGND -> GND
- R7 pad 1: /Conditioner1/Output -> /ADC1/Input
- R8 pad 1: /Conditioner1/+2.5V -> Net-(U1-+In_C)
- R9 pad 1: /Conditioner1/+2.5V -> Net-(U1-+In_C)
- R9 pad 2: AGND -> GND
- TP2 pad 1: /Conditioner1/+2.5V -> Net-(U1-+In_C)
- U1 pad 1: AGND -> GND
- U1 pad 10: /Conditioner1/+2.5V -> Net-(U1-+In_C)
- U1 pad 14: /Conditioner1/Output -> /ADC1/Input
- U1 pad 2: AGND -> GND
- U2 pad 3: AGND -> GND
- U3 pad 1: unconnected-(U3-Out_A-Pad1) -> GND
- U3 pad 10: /Conditioner1/+2.5V -> Net-(U3-+In_C)
- U3 pad 14: /Conditioner2/Output -> /ADC2/Input
- U3 pad 2: unconnected-(U3--In_A-Pad2) -> GND
- U3 pad 3: unconnected-(U3-+In_A-Pad3) -> Net-(U3-+In_A)
- U4 pad 1: unconnected-(U4-ADDR-Pad1) -> GND
- U4 pad 3: AGND -> GND
Routing:
- net GND: track 4.51 -> 56.6 mm, vias 0 -> 39
- net AGND: track 38.0 -> 0.00 mm, vias 15 -> 0
- net /ADC1/SDA: track 4.73 -> 35.7 mm
- net /ADC1/SCL: track 0.00 -> 30.7 mm
- net /ADC2/Input: track 0.00 -> 24.8 mm
- net +5V: track 58.6 -> 79.9 mm
- net /Conditioner1/+2.5V: track 21.0 -> 0.00 mm
- net Net-(U1-+In_C): track 0.00 -> 17.4 mm
- net Net-(U3-+In_A): track 0.00 -> 11.5 mm
- net /Conditioner1/Output: track 11.3 -> 0.00 mm
- net /ADC1/Input: track 0.00 -> 10.7 mm
- net Net-(U3-+In_C): track 0.00 -> 9.44 mm
- net /GPIO 22: track 0.00 -> 8.62 mm
- net /SDA: track 8.45 -> 0.00 mm
- net /GPIO 17: track 0.00 -> 8.42 mm
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- added copper zone on In2.Cu, net +12V
- added copper zone on In2.Cu, net -12V
- added copper zone on B.Cu, net GND
- added copper zone on F.Cu, net GND
- removed copper zone on In1.Cu, net AGND
Other:
- board size 70.9 x 39.9 mm -> 56.3 x 46.8 mm
- board text added: "Signal Conditioning & ADC Board Rev 1 Tyler Patterson"
