File: Hardware/modules/conditioner+adc module/conditioner+adc.kicad_sch (KiCad schematic)
At the start: 19 parts, among them J1 Conn_01x08_MountingPin, J2 Conn_01x08_MountingPin

Commit message: updates
Parts:
- removed J1, J2: Conn_01x08_MountingPin, Connector_PinHeader_2.54mm:PinHeader_1x08_P2.54mm_Vertical, symbol Connector_Generic_MountingPin:Conn_01x08_MountingPin
- removed R9: 1k, Resistor_SMD:R_0805_2012Metric_Pad1.20x1.40mm_HandSolder, symbol Device:R
- added C3, C4: 0.1 uF, Capacitor_SMD:C_0805_2012Metric_Pad1.18x1.45mm_HandSolder, symbol Device:C
- added C4_OPT1, C4_OPT2, C5_OPT1, C5_OPT2: C, Capacitor_SMD:C_0805_2012Metric_Pad1.18x1.45mm_HandSolder, symbol Device:C
- added D1, D2: LED, LED_SMD:LED_0805_2012Metric_Pad1.15x1.40mm_HandSolder, symbol Device:LED
- added J3: Conn_02x20_RaspberryPi_40Pin, 1Personal:CONN_RASPBERRYPI_40PIN_2x20, symbol Personal:Conn_02x20_RaspberryPi_40Pin
- added NT1: NetTie_2, NetTie:NetTie-2_SMD_Pad0.5mm, symbol Device:NetTie_2
- added P1-5k1, P2-5k1: TRIM_TS63Y, 1Personal:TRIM_TS63Y, symbol Custom:TRIM_TS63Y
- added R15, R17, R18, R20, R21, R22: 1k, Resistor_SMD:R_0805_2012Metric_Pad1.20x1.40mm_HandSolder, symbol Device:R
- added R19, R19_OPT1, R19_OPT2, R20_OPT1, R20_OPT2: R, Resistor_SMD:R_0805_2012Metric_Pad1.20x1.40mm_HandSolder, symbol Device:R
- added TP1, TP2: TestPoint, TestPoint:TestPoint_Pad_D2.0mm, symbol Connector:TestPoint
- added U2, U3: ADS1115, Package_SO:TSSOP-10_3x3mm_P0.5mm, symbol Analog_ADC:ADS1115IDGS
- R4: footprint Resistor_SMD:R_1206_3216Metric_Pad1.30x1.75mm_HandSolder -> Resistor_SMD:R_0603_1608Metric_Pad0.98x0.95mm_HandSolder
Connections:
- net GND: now also C3.1, J3.5 (Pin_5), NT1.2, R15.2; no longer C1.2, C2.1, R14.2, R3.2, R6.2, U1.2 (-In_A)
- net at R1.1, R2.1, U1.5 (+In_B): now also P2-5k1.1, TP1.1
- net at R10.1, R4.1, U1.10 (+In_C): now also P1-5k1.1, TP2.1
- net AGND: now reaches U1.1 (Out_A)
- net AGND: now also C1.2, C2.1, R14.2, R3.2, R6.2, U1.2 (-In_A), C4_OPT1.2, C4_OPT2.2, C5_OPT1.2, C5_OPT2.2, P1-5k1.2, P2-5k1.2, U2.1 (ADDR), U2.3 (GND), U3.3 (GND)
- net output renamed Cond1Output
- net Cond1Output: now also R19_OPT1.1
- new net: D2.1 (K), R19.1
- new net: C4.1, R19.2
- new net: D1.1 (K), R15.1
- new net: C4_OPT1.1, R19_OPT1.2, U2.4 (AIN0)
- new net: C5_OPT1.1, R20_OPT1.2, U2.5 (AIN1)
- new net: C4_OPT2.1, R19_OPT2.2, U3.4 (AIN0)
- new net: R20.2, U3.1 (ADDR), U3.10 (SCL)
- new net: R22.2, U3.2 (ALRT)
- new net: C5_OPT2.1, R20_OPT2.2, U3.5 (AIN1)
- new net: R21.2, U3.9 (SDA)
- new net +5V: C3.2, C4.2, D1.2 (A), D2.2 (A), J3.39 (Pin_39), R17.1, R18.1, R20.1, R21.1, R22.1, U2.8 (VDD), U3.8 (VDD)
- new net Cond2Output: R19_OPT2.1
- new net GNDA: NT1.1
- new net SCL: J3.3 (Pin_3), R17.2, U2.10 (SCL)
- new net SDA: J3.2 (Pin_2), R18.2, U2.9 (SDA)
- no-connect marks 10 -> 36
Other:
- moved on the sheet: C1, C2, R1, R10, R11, R12, R13, R14, R2, R3, R4, R5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

Commit message: p
Parts:
- removed C1, C2, C3, C4: 0.1 uF, Capacitor_SMD:C_0805_2012Metric_Pad1.18x1.45mm_HandSolder, symbol Device:C
- removed C4_OPT1, C4_OPT2, C5_OPT1, C5_OPT2: C, Capacitor_SMD:C_0805_2012Metric_Pad1.18x1.45mm_HandSolder, symbol Device:C
- removed D1, D2: LED, LED_SMD:LED_0805_2012Metric_Pad1.15x1.40mm_HandSolder, symbol Device:LED
- removed NT1: NetTie_2, NetTie:NetTie-2_SMD_Pad0.5mm, symbol Device:NetTie_2
- removed P1-5k1, P2-5k1: TRIM_TS63Y, 1Personal:TRIM_TS63Y, symbol Custom:TRIM_TS63Y
- removed R1: 3.3k, Resistor_SMD:R_0805_2012Metric_Pad1.20x1.40mm_HandSolder, symbol Device:R
- removed R10, R11, R12, R13, R14, R2, R7, R8: 10k, Resistor_SMD:R_0805_2012Metric_Pad1.20x1.40mm_HandSolder, symbol Device:R
- removed R15, R18, R20, R21, R22: 1k, Resistor_SMD:R_0805_2012Metric_Pad1.20x1.40mm_HandSolder, symbol Device:R
- removed R19, R19_OPT1, R19_OPT2, R20_OPT1, R20_OPT2: R, Resistor_SMD:R_0805_2012Metric_Pad1.20x1.40mm_HandSolder, symbol Device:R
- removed R3: 33.2, Resistor_SMD:R_0805_2012Metric_Pad1.20x1.40mm_HandSolder, symbol Device:R
- removed R4: 2.5K, Resistor_SMD:R_0603_1608Metric_Pad0.98x0.95mm_HandSolder, symbol Device:R
- removed R5: 130, Resistor_SMD:R_0603_1608Metric_Pad0.98x0.95mm_HandSolder, symbol Device:R
- removed R6: 1.58, Resistor_SMD:R_0603_1608Metric_Pad0.98x0.95mm_HandSolder, symbol Device:R
- removed TP1, TP2: TestPoint, TestPoint:TestPoint_Pad_D2.0mm, symbol Connector:TestPoint
- removed U1: ~, Package_SO:SOIC-14_3.9x8.7mm_P1.27mm, symbol Amplifier_Operational:_OPA4206
- removed U2, U3: ADS1115, Package_SO:TSSOP-10_3x3mm_P0.5mm, symbol Analog_ADC:ADS1115IDGS
- added C11, C13: 10 nF, symbol Custom:C
- added C12: 10 uF, symbol Custom:C
- added J2, J3: CONN_JST_1x2_1.25mmPitch, 1Personal:CONN_JST_1x2_1.25mmPitch, symbol Personal:CONN_JST_1x2_1.25mmPitch
- added P1-5k5: TRIM_TS63Y, 1Personal:TRIM_TS63Y, symbol Custom:TRIM_TS63Y
- added U5: IC_LinearRegulator_1-30VOutput, 1Personal:IC_LinearRegulator_1-30VOutput, symbol Personal:IC_LinearRegulator_1-30VOutput
- R17: value 1k -> 3.3k; footprint Resistor_SMD:R_0805_2012Metric_Pad1.20x1.40mm_HandSolder -> (none)
- renumbered J3 to J1
Connections:
- net +5V: no longer R17.1
- net GND: now also C11.2, J2.2
- net SCL: no longer R17.2
- new net: C11.1, U5.6 (NR/SS)
- new net: C12.1, C13.1, R17.1, U5.1 (OUT)
- new net: C13.2, U5.2 (FB)
- new net: P1-5k5.1, R17.2
- new net: J2.1, U5.5 (EN), U5.8 (IN)
- no-connect marks 36 -> 30
Other:
- added sheet ADC1 (ADC1.kicad_sch)
- added sheet ADC2 (ADC1.kicad_sch)
- added sheet Conditioner1 (Conditioner1.kicad_sch)
- added sheet Conditioner2 (Conditioner1.kicad_sch)

Commit message: p
Parts:
- removed J3: CONN_JST_1x2_1.25mmPitch, 1Personal:CONN_JST_1x2_1.25mmPitch, symbol Personal:CONN_JST_1x2_1.25mmPitch
- added R18: 10k, Resistor_SMD:R_0805_2012Metric_Pad1.20x1.40mm_HandSolder, symbol Device:R
- R17: value 3.3k -> 10k; footprint (none) -> Resistor_SMD:R_0805_2012Metric_Pad1.20x1.40mm_HandSolder
Connections:
- net at C12.1, C13.1, U5.1 (OUT): now also R18.1; no longer R17.1
- net at C13.2, U5.2 (FB): now also P1-5k5.2
- net GNDA: now reaches C12.2
- new net: R17.1, R18.2
Other:
- moved on the sheet: C12, P1-5k5

Commit message: p
Parts:
- removed C11, C13: 10 nF, symbol Custom:C
- removed C12: 10 uF, symbol Custom:C
- removed P1-5k5: TRIM_TS63Y, 1Personal:TRIM_TS63Y, symbol Custom:TRIM_TS63Y
- removed R17, R18: 10k, Resistor_SMD:R_0805_2012Metric_Pad1.20x1.40mm_HandSolder, symbol Device:R
- added C12, C13: 10 nF, symbol Device:C
- added C14: 10 uF, symbol Device:C
- added J2, J3: CONN_JST_1x2_1.25mmPitch, 1Personal:CONN_JST_1x2_1.25mmPitch, symbol Personal:CONN_JST_1x2_1.25mmPitch
- added R23: 51.1k, Resistor_SMD:R_0805_2012Metric_Pad1.20x1.40mm_HandSolder, symbol Device:R
- added RV1: 5k, 1Personal:TRIM_TS63Y, symbol Device:R_Potentiometer_US
- renumbered J2 to J1, J1 to J4
Connections:
- net Conditioner1/Input: now also J3.2
- net Conditioner2/Input: now also J2.2
- net GND: now also U5.9 (POWERPAD), U5.9_2 (POWERPAD__2), U5.9_4 (POWERPAD__4), C12.2
- net at U5.6 (NR/SS): now also C12.1
- net at U5.1 (OUT): now also C13.1, C14.1, R23.1
- net at U5.2 (FB): now also C13.2, R23.2, RV1.1
- net AGND: now reaches U5.4 (GND)
- net AGND: now also U5.9_1 (POWERPAD__1), U5.9_3 (POWERPAD__3), C14.2, J2.1, J3.1, RV1.2
- no-connect marks 30 -> 32
Other:
- sheet ADC2: file ADC1.kicad_sch -> ADC2.kicad_sch
- sheet Conditioner1 ports: added +12V, +2.5V, -12V; removed none
- sheet Conditioner2: file Conditioner1.kicad_sch -> Conditioner2.kicad_sch
- sheet Conditioner2 ports: added +12V, +2.5V, -12V; removed none

Commit message: p
Parts:
- removed C12, C13: 10 nF, symbol Device:C
- removed C14: 10 uF, symbol Device:C
- removed RV1: 5k, 1Personal:TRIM_TS63Y, symbol Device:R_Potentiometer_US
- removed U5: IC_LinearRegulator_1-30VOutput, 1Personal:IC_LinearRegulator_1-30VOutput, symbol Personal:IC_LinearRegulator_1-30VOutput
- added J5: Conn_01x06, 1Personal:CONN_JST_1x6_1.25mmPitch, symbol Connector_Generic:Conn_01x06
- added J6: Conn_01x03, 1Personal:CONN_JST_1x3_1.25mmPitch, symbol Connector_Generic:Conn_01x03
- added R24: 10k, Resistor_SMD:R_0805_2012Metric_Pad1.20x1.40mm_HandSolder, symbol Device:R
- R23: value 51.1k -> 10k
Connections:
- net AGND is gone; now on net GND: J2.1, J3.1
- net SCL is gone; now on net ADC1/SCL: J4.3 (Pin_3)
- net SDA is gone; now on net ADC1/SDA: J4.2 (Pin_2)
- net +5V: now also R23.2, J5.6 (Pin_6), R24.1
- net ADC1/SCL: now also R23.1
- net ADC1/SDA: now also R24.2
- net GND: now also J5.1 (Pin_1), J6.1 (Pin_1); no longer J1.2
- net GPIO 23: now reaches J4.33 (Pin_33)
- net GPIO 23: now also J5.3 (Pin_3)
- net UART RX: now reaches J4.36 (Pin_36)
- net UART RX: now also J6.2 (Pin_2)
- net UART TX: now reaches J4.37 (Pin_37)
- net UART TX: now also J6.3 (Pin_3)
- net GPIO 17: now reaches J4.6 (Pin_6)
- net GPIO 17: now also J5.5 (Pin_5)
- net GPIO 27: now reaches J4.7 (Pin_7)
- net GPIO 27: now also J5.4 (Pin_4)
- net GPIO 22: now reaches J4.8 (Pin_8)
- net GPIO 22: now also J5.2 (Pin_2)
- net +12V: now reaches J1.1
- new net -12V: J1.2
- no-connect marks 32 -> 24
